File: PCB/Sheet/Sheet.kicad_sch (KiCad schematic)
At the start: 2 parts, among them U1 74LVC2G74, U2 SN74LVC1G00DBV

Commit message: Update Sheet.kicad_sch
Parts:
- removed U1: 74LVC2G74, symbol 74xGxx:74LVC2G74
- added U1: 74LVC1G04, symbol 74xGxx:74LVC1G04
- added U10, U11, U12, U13, U14, U15, U6: SN74LVC1G00DBV, Package_TO_SOT_SMD:SOT-23-5, symbol 74xGxx:SN74LVC1G00DBV
- added U3, U4, U5, U7, U8, U9: 74AUP1G08, symbol 74xGxx:74AUP1G08
Connections:
- net at U2.1: now also U5.4, U8.4
- net Rerouting logic: now reaches U2.3 (GND)
- net Rerouting logic: now also U1.3 (GND), U3.3 (GND), U4.3 (GND), U5.3 (GND), U6.3 (GND)
- net at U2.4: now also U3.1
- net at U2.5 (VCC): now also U1.5 (VCC), U10.5 (VCC), U11.5 (VCC), U12.5 (VCC), U13.5 (VCC), U14.5 (VCC), U15.5 (VCC), U3.5 (VCC), U4.5 (VCC), U5.5 (VCC), U6.5 (VCC), U7.5 (VCC), U8.5 (VCC), U9.5 (VCC)
- new net: U3.4, U7.1, U8.1, U9.1, U9.4
- new net: U10.4, U7.2
- new net: U7.3 (GND), U8.3 (GND), U9.3 (GND)
- new net: U4.4, U6.1, U7.4
- new net: U10.2, U11.1
- new net: U10.3 (GND), U11.3 (GND), U12.3 (GND), U13.3 (GND), U14.3 (GND), U15.3 (GND)
- new net: U14.2, U15.1
- new net: U14.4, U9.2
- new net: U11.2, U13.2, U15.2
- new net: U5.1, U6.4
- new net: U12.2, U13.1
- new net: U12.4, U8.2
- new net: U1.4, U4.2
Other:
- company: (none) -> Dexter R. Shepherd
- title: (none) -> TacSheet flexible sensor

Commit message: Update Sheet.kicad_sch
Parts:
- added L1: DelayLine, symbol Device:DelayLine
- added R1: R, symbol Device:R
- added U16, U17, U18, U19: 74AUP1G32, symbol 74xGxx:74AUP1G32
- added U20: 74LVC1G66, symbol 74xGxx:74LVC1G66
Connections:
- net Data in B: now also U12.1, U18.2
- net at U7.2: now also U10.2, U11.4, U16.1; no longer U10.4
- net at U1.5 (VCC), U10.5 (VCC), U11.5 (VCC)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: now also R1.1, U16.5 (VCC), U17.5 (VCC), U18.5 (VCC), U19.5 (VCC)
- net at U10.1: now also U19.2
- net at U11.1: now also U10.4; no longer U10.2
- net at U14.1: now also U18.1
- net at U14.2: now also U15.4, U9.2, U17.2; no longer U15.1
- net at U14.4: now also U15.1; no longer U9.2
- net at U5.2: now also U3.2, U4.1
- net at U12.2: now also U13.4, U8.2, U16.2; no longer U13.1
- net at U12.4: now also U13.1; no longer U8.2
- new net: L1.1, U20.2
- new net: R1.2, U20.1
- new net: U19.4, U20.4
- new net: U16.3 (GND), U17.3 (GND)
- new net: U16.4, U17.1
- new net: U18.4, U19.1
- new net: U18.3 (GND), U19.3 (GND)

Commit message: schematics
Parts:
- removed L1: DelayLine, symbol Device:DelayLine
- removed U1: 74LVC1G04, symbol 74xGxx:74LVC1G04
- removed U10, U11, U12, U13, U14, U15, U2, U6: SN74LVC1G00DBV, Package_TO_SOT_SMD:SOT-23-5, symbol 74xGxx:SN74LVC1G00DBV
- removed U16, U17, U18, U19: 74AUP1G32, symbol 74xGxx:74AUP1G32
- removed U20: 74LVC1G66, symbol 74xGxx:74LVC1G66
- removed U3, U4, U5, U7, U8, U9: 74AUP1G08, symbol 74xGxx:74AUP1G08
- added C1, C2: C, symbol Device:C
- added R2: R, symbol Device:R
- added U1: ATtiny85-20S, Package_SO:SOIC-8W_5.3x5.3mm_P1.27mm, symbol MCU_Microchip_ATtiny:ATtiny85-20S
- added U2: MAX3485, symbol Interface_UART:MAX3485
- added U3: ATtiny1616-M, Package_DFN_QFN:VQFN-20-1EP_3x3mm_P0.4mm_EP1.7x1.7mm, symbol MCU_Microchip_ATtiny:ATtiny1616-M
- added U4: ~, symbol sensors:ADXL335
- added U5: MCP9700Ax-ETT, Package_TO_SOT_SMD:SOT-23, symbol Sensor_Temperature:MCP9700Ax-ETT
Connections:
- net at R1.1: now also C1.2, U1.2 (XTAL1/PB3), U1.4 (GND), U2.5 (GND)
- net 100nF: now reaches R1.2
- net 100nF: now also C1.1, U1.8 (VCC), U2.8 (VCC)
- new net: U1.5 (AREF/PB0), U2.4 (DI)
- new net: U1.6 (PB1), U2.1 (RO)
- new net: U1.7 (PB2), U2.2 (~{RE}), U2.3 (DE)
- new net: U3.10 (PB4), U4. (vcc)
- new net: U3.11 (PB3), U4. (vcc)
- new net: C2.2, R2.2, U3.21 (GND), U3.3 (GND), U3.8 (PA7), U4. (vcc), U5.3 (GND)
- new net: C2.1, R2.1, U3.4 (VCC), U4. (vcc), U5.1 (V_{DD})
- new net: U3.7 (PA6), U5.2 (V_{OUT})
- new net: U3.9 (PB5), U4. (vcc)
- new net BUS A: U2.6 (A)
- new net Bus B: U2.7 (B)

Commit message: designs
Parts:
- removed C1: C, symbol Device:C
- removed U1: ATtiny85-20S, Package_SO:SOIC-8W_5.3x5.3mm_P1.27mm, symbol MCU_Microchip_ATtiny:ATtiny85-20S
- removed U2: MAX3485, symbol Interface_UART:MAX3485
- removed U5: MCP9700Ax-ETT, Package_TO_SOT_SMD:SOT-23, symbol Sensor_Temperature:MCP9700Ax-ETT
- added R3, R4, R5, R6: R, symbol Device:R
- added U1: MCP9700Ax-ELT, Package_TO_SOT_SMD:SOT-353_SC-70-5, symbol Sensor_Temperature:MCP9700Ax-ELT
- added U2: MCP2562-E-MF, Package_DFN_QFN:DFN-8-1EP_3x3mm_P0.65mm_EP1.55x2.4mm, symbol Interface_CAN_LIN:MCP2562-E-MF
- added U5: MCP2515-xSO, Package_SO:SOIC-18W_7.5x11.6mm_P1.27mm, symbol Interface_CAN_LIN:MCP2515-xSO
Connections:
- net 100nF: no longer R1.2
- net at R1.1: now also C2.1, R2.1, U3.4 (VCC), U4. (vcc), R3.1, R4.1, R5.1, R6.1, U1.4 (V_{DD}), U2.3 (VDD), U5.18 (VDD)
- net at U3.1 (PA2): now also U5.15 (SO)
- net at U3.14 (PB0): now also C2.2, R1.2, R2.2, U3.16 (PC1), U3.17 (PC2), U3.18 (PC3), U3.21 (GND), U3.3 (GND), U3.6 (PA5), U3.8 (PA7), U4. (vcc), R3.2, R4.2, R5.2, R6.2, U1.2 (GND), U2.2 (VSS), U5.9 (VSS)
- net at U3.15 (PC0): now also U5.12 (~{INT})
- net at U3.2 (PA3): now also U5.13 (SCK)
- net at U3.20 (PA1): now also U5.14 (SI)
- net at U3.5 (PA4): now also U5.16 (~{CS})
- net at U3.7 (PA6): now also U1.3 (V_{OUT})
- new net: U2.1 (TXD), U5.1 (TXCAN)
- new net: U2.4 (RXD), U5.2 (RXCAN)
- now unconnected: U4. (vcc), U4. (vcc)

Commit message: PCB design
Parts:
- removed U5: MCP2515-xSO, Package_SO:SOIC-18W_7.5x11.6mm_P1.27mm, symbol Interface_CAN_LIN:MCP2515-xSO
- added D1: LED, symbol Device:LED
- added D2: D, symbol Device:D
- added R7: R, symbol Device:R
- added U6: MCP2515-xST, Package_SO:TSSOP-20_4.4x6.5mm_P0.65mm, symbol Interface_CAN_LIN:MCP2515-xST
Connections:
- net at C2.2, R1.2, R2.2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: now also D2.2 (A), U6.10 (VSS)
- net at C2.1, R1.1, R2.1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: now also R7.1, U6.20 (VDD)
- net at U3.1 (PA2): now also U6.17 (SO)
- net at U3.15 (PC0): now also U6.6 (NC)
- net at U3.2 (PA3): now also U6.14 (SCK)
- net at U3.20 (PA1): now also U6.16 (SI)
- net at U3.5 (PA4): now also U6.18 (~{CS})
- net at U2.1 (TXD): now also U6.1 (TXCAN)
- net at U2.4 (RXD): now also U6.2 (RXCAN)
- new net: D1.1 (K), D2.1 (K)
- new net: D1.2 (A), R7.2
Changed lines of the file:
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@@
   (junction (at 166.37 71.12) (diameter 0) (color 0 0 0 0)
   )
+  (junction (at 80.01 69.85) (diameter 0) (color 0 0 0 0)
+  )
   (junction (at 80.01 34.29) (diameter 0) (color 0 0 0 0)
   )
@@
   (junction (at 80.01 64.77) (diameter 0) (color 0 0 0 0)
   )
+  (junction (at 148.59 46.99) (diameter 0) (color 0 0 0 0)
+  )
   (junction (at 119.38 115.57) (diameter 0) (color 0 0 0 0)
   )
-  (junction (at 148.59 46.99) (diameter 0) (color 0 0 0 0)
-  )
   (junction (at 148.59 19.05) (diameter 0) (color 0 0 0 0)
   )
@@
   (junction (at 144.78 19.05) (diameter 0) (color 0 0 0 0)
   )
+  (junction (at 80.01 27.94) (diameter 0) (color 0 0 0 0)
+  )
   (junction (at 148.59 41.91) (diameter 0) (color 0 0 0 0)
   )
@@
   (junction (at 114.3 19.05) (diameter 0) (color 0 0 0 0)
   )
+  (wire (pts (xy 80.01 69.85) (xy 80.01 64.77))
+    (stroke (width 0) (type default))
+  )
   (wire (pts (xy 82.55 46.99) (xy 82.55 44.45))
     (stroke (width 0) (type default))
@@
     (stroke (width 0) (type default))
   )
+  (wire (pts (xy 69.85 54.61) (xy 69.85 58.42))
+    (stroke (width 0) (type default))
+  )
   (wire (pts (xy 86.36 46.99) (xy 91.44 46.99))
     (stroke (width 0) (type default))
   )
+  (wire (pts (xy 106.68 95.25) (xy 92.71 95.25))
+    (stroke (width 0) (type default))
+  )
   (wire (pts (xy 148.59 21.59) (xy 148.59 19.05))
     (stroke (width 0) (type default))
@@
     (stroke (width 0) (type default))
   )
-  (wire (pts (xy 134.62 95.25) (xy 92.71 95.25))
-    (stroke (width 0) (type default))
-  )
   (wire (pts (xy 82.55 46.99) (xy 86.36 46.99))
     (stroke (width 0) (type default))
@@
     (stroke (width 0) (type default))
   )
+  (wire (pts (xy 69.85 66.04) (xy 69.85 69.85))
+    (stroke (width 0) (type default))
+  )
   (wire (pts (xy 167.64 31.75) (xy 171.45 31.75))
     (stroke (width 0) (type default))
@@
     (stroke (width 0) (type default))
   )
+  (wire (pts (xy 119.38 115.57) (xy 166.37 115.57))
+    (stroke (width 0) (type default))
+  )
+  (wire (pts (xy 68.58 27.94) (xy 80.01 27.94))
+    (stroke (width 0) (type default))
+  )
   (wire (pts (xy 99.06 52.07) (xy 86.36 52.07))
     (stroke (width 0) (type default))
@@
     (stroke (width 0) (type default))
   )
-  (wire (pts (xy 119.38 115.57) (xy 166.37 115.57))
+  (wire (pts (xy 80.01 115.57) (xy 119.38 115.57))
     (stroke (width 0) (type default))
   )
@@
     (stroke (width 0) (type default))
   )
-  (wire (pts (xy 80.01 115.57) (xy 80.01 64.77))
+  (wire (pts (xy 80.01 69.85) (xy 80.01 115.57))
     (stroke (width 0) (type default))
   )
@@
     (stroke (width 0) (type default))
   )
+  (wire (pts (xy 80.01 27.94) (xy 80.01 34.29))
+    (stroke (width 0) (type default))
+  )
   (wire (pts (xy 133.35 31.75) (xy 133.35 67.31))
     (stroke (width 0) (type default))
   )
+  (wire (pts (xy 68.58 54.61) (xy 69.85 54.61))
+    (stroke (width 0) (type default))
+  )
   (wire (pts (xy 100.33 71.12) (xy 100.33 82.55))
     (stroke (width 0) (type default))
@@
     (stroke (width 0) (type default))
   )
+  (wire (pts (xy 72.39 69.85) (xy 69.85 69.85))
+    (stroke (width 0) (type default))
+  )
   (wire (pts (xy 129.54 31.75) (xy 133.35 31.75))
     (stroke (width 0) (type default))
@@
     (stroke (width 0) (type default))
   )
-  (wire (pts (xy 119.38 115.57) (xy 80.01 115.57))
+  (wire (pts (xy 68.58 46.99) (xy 68.58 27.94))
     (stroke (width 0) (type default))
   )
@@
     (stroke (width 0) (type default))
   )
-  (wire (pts (xy 80.01 19.05) (xy 80.01 34.29))
+  (wire (pts (xy 80.01 19.05) (xy 80.01 27.94))
     (stroke (width 0) (type default))
   )
@@
     )
   )
+  (symbol (lib_id "Interface_CAN_LIN:MCP2515-xST") (at 119.38 95.25 0) (unit 1)
+    (in_bom yes) (on_board yes) (dnp no) (fields_autoplaced)
+    (property "Reference" "U6" (at 121.5741 72.39 0)
+      (effects (font (size 1.27 1.27)) (justify left))
+    )
+    (property "Value" "MCP2515-xST" (at 121.5741 74.93 0)
+      (effects (font (size 1.27 1.27)) (justify left))
+    )
+    (property "Footprint" "Package_SO:TSSOP-20_4.4x6.5mm_P0.65mm" (at 119.38 118.11 0)
+      (effects (font (size 1.27 1.27) italic) hide)
+    )
+    (property "Datasheet" "http://ww1.microchip.com/downloads/en/DeviceDoc/21801e.pdf" (at 121.92 115.57 0)
+      (effects (font (size 1.27 1.27)) hide)
+    )
+    (pin "8")
+    (pin "9")
+    (pin "2")
+    (pin "15")
+    (pin "14")
+    (pin "6")
+    (pin "19")
+    (pin "17")
+    (pin "7")
+    (pin "13")
+    (pin "12")
+    (pin "3")
+    (pin "11")
+    (pin "5")
+    (pin "1")
+    (pin "10")
+    (pin "18")
+    (pin "20")
+    (pin "16")
+    (pin "4")
+    (instances
+      (project "Sheet"
+        (path "/3799ba30-20d0-42d8-8664-7c6f9d1278f6"
+          (reference "U6") (unit 1)
+        )
+      )
+    )
+  )
   (symbol (lib_id "Device:R") (at 148.59 25.4 0) (unit 1)
     (in_bom yes) (on_board yes) (dnp no) (fields_autoplaced)
@@
     )
   )
+  (symbol (lib_id "Device:LED") (at 69.85 62.23 90) (unit 1)
+    (in_bom yes) (on_board yes) (dnp no)
+    (property "Reference" "D1" (at 67.31 65.0875 90)
+      (effects (font (size 1.27 1.27)) (justify left))
+    )
+    (property "Value" "LED" (at 67.31 62.5475 90)
+      (effects (font (size 1.27 1.27)) (justify left))
+    )
+    (property "Footprint" "" (at 69.85 62.23 0)
+      (effects (font (size 1.27 1.27)) hide)
+    )
+    (property "Datasheet" "~" (at 69.85 62.23 0)
+      (effects (font (size 1.27 1.27)) hide)
+    )
+    (pin "1")
+    (pin "2")
+    (instances
+      (project "Sheet"
+        (path "/3799ba30-20d0-42d8-8664-7c6f9d1278f6"
+          (reference "D1") (unit 1)
+        )
+      )
+    )
+  )
   (symbol (lib_id "Device:R") (at 91.44 50.8 0) (unit 1)
     (in_bom yes) (on_board yes) (dnp no) (fields_autoplaced)
@@
     )
   )
-  (symbol (lib_id "Interface_CAN_LIN:MCP2515-xSO") (at 119.38 95.25 0) (unit 1)
-    (in_bom yes) (on_board yes) (dnp no) (fields_autoplaced)
-    (property "Reference" "U5" (at 121.5741 72.39 0)
-      (effects (font (size 1.27 1.27)) (justify left))
-    )
-    (property "Value" "MCP2515-xSO" (at 121.5741 74.93 0)
-      (effects (font (size 1.27 1.27)) (justify left))
-    )
-    (property "Footprint" "Package_SO:SOIC-18W_7.5x11.6mm_P1.27mm" (at 119.38 118.11 0)
-      (effects (font (size 1.27 1.27) italic) hide)
-    )
-    (property "Datasheet" "http://ww1.microchip.com/downloads/en/DeviceDoc/21801e.pdf" (at 121.92 115.57 0)
-      (effects (font (size 1.27 1.27)) hide)
-    )
-    (pin "9")
-    (pin "12")
-    (pin "11")
-    (pin "4")
-    (pin "8")
-    (pin "5")
-    (pin "2")
-    (pin "17")
-    (pin "7")
-    (pin "18")
-    (pin "3")
-    (pin "16")
-    (pin "1")
-    (pin "14")
-    (pin "6")
-    (pin "10")
-    (pin "13")
-    (pin "15")
-    (instances
-      (project "Sheet"
-        (path "/3799ba30-20d0-42d8-8664-7c6f9d1278f6"
-          (reference "U5") (unit 1)
-        )
-      )
+  (symbol (lib_id "Device:R") (at 68.58 50.8 0) (unit 1)
+    (in_bom yes) (on_board yes) (dnp no) (fields_autoplaced)
+    (property "Reference" "R7" (at 71.12 49.53 0)
+      (effects (font (size 1.27 1.27)) (justify left))
+    )
+    (property "Value" "R" (at 71.12 52.07 0)
+      (effects (font (size 1.27 1.27)) (justify left))
+    )
+    (property "Footprint" "" (at 66.802 50.8 90)
+      (effects (font (size 1.27 1.27)) hide)
+    )
+    (property "Datasheet" "~" (at 68.58 50.8 0)
+      (effects (font (size 1.27 1.27)) hide)
+    )
+    (pin "1")
+    (pin "2")
+    (instances
+      (project "Sheet"
+        (path "/3799ba30-20d0-42d8-8664-7c6f9d1278f6"
+          (reference "R7") (unit 1)
+        )
+      )
+    )
+  )
+  (symbol (lib_id "Device:D") (at 76.2 69.85 0) (unit 1)
+    (in_bom yes) (on_board yes) (dnp no) (fields_autoplaced)
+    (property "Reference" "D2" (at 76.2 63.5 0)
+      (effects (font (size 1.27 1.27)))
+    )
+    (property "Value" "D" (at 76.2 66.04 0)
+      (effects (font (size 1.27 1.27)))
+    )
+    (property "Footprint" "" (at 76.2 69.85 0)
+      (effects (font (size 1.27 1.27)) hide)
+    )
+    (property "Datasheet" "~" (at 76.2 69.85 0)
+      (effects (font (size 1.27 1.27)) hide)
+    )
+    (property "Sim.Device" "D" (at 76.2 69.85 0)
+      (effects (font (size 1.27 1.27)) hide)
+    )
+    (property "Sim.Pins" "1=K 2=A" (at 76.2 69.85 0)
+      (effects (font (size 1.27 1.27)) hide)
+    )
+    (pin "1")
+    (pin "2")
+    (instances
+      (project "Sheet"
+        (path "/3799ba30-20d0-42d8-8664-7c6f9d1278f6"
+          (reference "D2") (unit 1)
+        )
+      )

Commit message: updates
Other:
- moved on the sheet: C2, D1, D2, R1, R2, R3, R4, R5, R6, R7, U1, U2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

Commit message: PCB updates
Parts:
- added R8: 120 R, symbol Device:R_US
- added Y1: 8Hz, symbol Device:Crystal
Connections:
- net at U6.8 (OSC2): now also Y1.2
- net at U6.9 (OSC1): now also Y1.1
- net at U2.6 (CANL): now also R8.2
- net at U2.7 (CANH): now also R8.1
Changed lines of the file:
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@@
   (junction (at 161.29 106.68) (diameter 0) (color 0 0 0 0)
   )
+  (junction (at 267.97 125.73) (diameter 0) (color 0 0 0 0)
+  )
   (junction (at 229.87 88.9) (diameter 0) (color 0 0 0 0)
   )
@@
   (junction (at 226.06 60.96) (diameter 0) (color 0 0 0 0)
   )
+  (junction (at 267.97 120.65) (diameter 0) (color 0 0 0 0)
+  )
   (junction (at 161.29 69.85) (diameter 0) (color 0 0 0 0)
   )
@@
   (junction (at 195.58 60.96) (diameter 0) (color 0 0 0 0)
   )
+  (wire (pts (xy 167.64 147.32) (xy 167.64 143.51))
+    (stroke (width 0) (type default))
+  )
   (wire (pts (xy 161.29 111.76) (xy 161.29 106.68))
     (stroke (width 0) (type default))
@@
     (stroke (width 0) (type default))
   )
+  (wire (pts (xy 175.26 143.51) (xy 185.42 143.51))
+    (stroke (width 0) (type default))
+  )
   (wire (pts (xy 170.18 76.2) (xy 161.29 76.2))
     (stroke (width 0) (type default))
@@
     (stroke (width 0) (type default))
   )
+  (wire (pts (xy 260.35 120.65) (xy 267.97 120.65))
+    (stroke (width 0) (type default))
+  )
   (wire (pts (xy 181.61 124.46) (xy 185.42 124.46))
     (stroke (width 0) (type default))
@@
     (stroke (width 0) (type default))
   )
+  (wire (pts (xy 175.26 147.32) (xy 167.64 147.32))
+    (stroke (width 0) (type default))
+  )
   (wire (pts (xy 167.64 93.98) (xy 167.64 96.52))
     (stroke (width 0) (type default))
@@
     (stroke (width 0) (type default))
   )
-  (wire (pts (xy 260.35 125.73) (xy 274.32 125.73))
+  (wire (pts (xy 260.35 125.73) (xy 267.97 125.73))
     (stroke (width 0) (type default))
   )
@@
     (stroke (width 0) (type default))
   )
+  (wire (pts (xy 267.97 125.73) (xy 274.32 125.73))
+    (stroke (width 0) (type default))
+  )
   (wire (pts (xy 220.98 101.6) (xy 210.82 101.6))
     (stroke (width 0) (type default))
@@
     (stroke (width 0) (type default))
   )
+  (wire (pts (xy 267.97 118.11) (xy 267.97 120.65))
+    (stroke (width 0) (type default))
+  )
   (wire (pts (xy 214.63 73.66) (xy 214.63 109.22))
     (stroke (width 0) (type default))
@@
     (stroke (width 0) (type default))
   )
+  (wire (pts (xy 267.97 120.65) (xy 274.32 120.65))
+    (stroke (width 0) (type default))
+  )
   (wire (pts (xy 153.67 111.76) (xy 151.13 111.76))
     (stroke (width 0) (type default))
   )
+  (wire (pts (xy 185.42 144.78) (xy 175.26 144.78))
+    (stroke (width 0) (type default))
+  )
   (wire (pts (xy 210.82 73.66) (xy 214.63 73.66))
     (stroke (width 0) (type default))
@@
     (stroke (width 0) (type default))
   )
+  (wire (pts (xy 185.42 143.51) (xy 185.42 142.24))
+    (stroke (width 0) (type default))
+  )
   (wire (pts (xy 210.82 86.36) (xy 210.82 88.9))
     (stroke (width 0) (type default))
@@
     (stroke (width 0) (type default))
   )
+  (wire (pts (xy 175.26 144.78) (xy 175.26 147.32))
+    (stroke (width 0) (type default))
+  )
   (wire (pts (xy 215.9 92.71) (xy 215.9 96.52))
     (stroke (width 0) (type default))
@@
   )
   (wire (pts (xy 226.06 73.66) (xy 226.06 78.74))
-    (stroke (width 0) (type default))
-  )
-  (wire (pts (xy 260.35 120.65) (xy 274.32 120.65))
     (stroke (width 0) (type default))
   )
@@
     (effects (font (size 1.27 1.27)) (justify left bottom))
   )
+  (symbol (lib_id "Device:Crystal") (at 171.45 143.51 0) (unit 1)
+    (in_bom yes) (on_board yes) (dnp no) (fields_autoplaced)
+    (property "Reference" "Y1" (at 171.45 135.89 0)
+      (effects (font (size 1.27 1.27)))
+    )
+    (property "Value" "8Hz" (at 171.45 138.43 0)
+      (effects (font (size 1.27 1.27)))
+    )
+    (property "Footprint" "" (at 171.45 143.51 0)
+      (effects (font (size 1.27 1.27)) hide)
+    )
+    (property "Datasheet" "~" (at 171.45 143.51 0)
+      (effects (font (size 1.27 1.27)) hide)
+    )
+    (pin "2")
+    (pin "1")
+    (instances
+      (project "Sheet"
+        (path "/3799ba30-20d0-42d8-8664-7c6f9d1278f6"
+          (reference "Y1") (unit 1)
+        )
+      )
+    )
+  )
+  (symbol (lib_id "Device:R_US") (at 267.97 121.92 0) (unit 1)
+    (in_bom yes) (on_board yes) (dnp no) (fields_autoplaced)
+    (property "Reference" "R8" (at 270.51 120.65 0)
+      (effects (font (size 1.27 1.27)) (justify left))
+    )
+    (property "Value" "120 R" (at 270.51 123.19 0)
+      (effects (font (size 1.27 1.27)) (justify left))
+    )
+    (property "Footprint" "" (at 268.986 122.174 90)
+      (effects (font (size 1.27 1.27)) hide)
+    )
+    (property "Datasheet" "~" (at 267.97 121.92 0)
+      (effects (font (size 1.27 1.27)) hide)
+    )
+    (pin "1")
+    (pin "2")
+    (instances
+      (project "Sheet"
+        (path "/3799ba30-20d0-42d8-8664-7c6f9d1278f6"
+          (reference "R8") (unit 1)
+        )
+      )
+    )
+  )
   (symbol (lib_id "Sensor_Temperature:MCP9700Ax-ELT") (at 260.35 73.66 90) (unit 1)
