File: PCB/Sheet/Sheet.kicad_sch (KiCad schematic)
At the start: 19 parts, among them U1 MCP9700Ax-ELT, U2 MCP2562-E-MF, U3 ATtiny1616-M, U5 CD74HC4067SM, U6 MCP2515-xST, Y1 8Hz

Commit message: files
Parts:
- added C1, C3, C4: C, symbol Device:C
- added MK1: Microphone, symbol Device:Microphone
- added R10, R11, R12, R9: R, symbol Device:R
- added U7, U8: DRV5055A1xDBZxQ1, Package_TO_SOT_SMD:SOT-23, symbol Sensor_Magnetic:DRV5055A1xDBZxQ1
- Y1: value 8Hz -> 8Mhz
Connections:
- net at U1.4 (V_{DD}), U2.3 (VDD), U2.5 (Vio)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: now also U6.19 (~{RESET}), C1.2, C3.1, R9.2, U7.1 (VCC), U8.1 (VCC)
- net at C2.2, R1.1, R2.1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: now also C1.1, C3.2, C4.2, MK1.1 (-), R10.1, R11.1, R12.1, U7.3 (GND), U8.3 (GND)
- net at U5.18 (I13): now also U4. (vcc)
- net at U5.23 (I8): now also U7.2 (OUT); no longer U4. (vcc)
- net at U5.5 (I4): now also R10.2
- net at U5.6 (I3): now also C4.1, MK1.2 (+), R9.1
- net at U5.7 (I2): now also R11.2
- net at U5.8 (I1): now also R12.2
- net at U5.9 (I0): now also U8.2 (OUT)

Commit message: reorg
Parts:
- removed U4: ~, symbol sensors:ADXL335
- added C10, C11, C12, C13: 0.1uF, Capacitor_SMD:C_0603_1608Metric, symbol Device:C_Small
- added C14: 220pF, Capacitor_SMD:C_0603_1608Metric, symbol Device:C_Small
- added C5, C6, C7: C, symbol Device:C
- added C8: 4.7uF, Capacitor_SMD:C_0603_1608Metric, symbol Device:C_Small
- added C9: 10uF, Capacitor_SMD:C_0603_1608Metric, symbol Device:C_Small
- added J1: Conn_01x08, Connector_PinHeader_2.54mm:PinHeader_1x08_P2.54mm_Horizontal, symbol Connector_Generic:Conn_01x08
- added R13, R14, R15, R16, R17, R18, R19, R20, R21, R22, R23, R24, R25, R26, R27, R28, R29, R30, R31, R32, R33, R34, R35, R36, R37, R38, R39: R, symbol Device:R
- added R40: 1k, Resistor_SMD:R_0603_1608Metric, symbol Device:R_Small_US
- added R41, R42, R43, R44: 4.7k, Resistor_SMD:R_0603_1608Metric, symbol Device:R_Small_US
- added U10, U11, U9: ADS7830, Package_SO:TSSOP-16_4.4x5mm_P0.65mm, symbol Analog_DAC:ADS7830
- added U12: MPU-6050, Sensor_Motion:InvenSense_QFN-24_4x4mm_P0.5mm, symbol Sensor_Motion:MPU-6050
- added U4: AP2112K-3.3, Package_TO_SOT_SMD:SOT-23-5, symbol Regulator_Linear:AP2112K-3.3
Connections:
- net at C1.2, C3.1, R9.2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: now also C5.1, C6.1, C7.1, R37.1, R38.1, R39.1, U10.16 (VDD), U11.16 (VDD), U9.16 (VDD)
- net at U3.13 (PB1): now also U10.15 (SDA), U11.15 (SDA), U9.15 (SDA)
- net at U3.14 (PB0): now also U10.14 (SCL), U11.14 (SCL), U9.14 (SCL)
- net at C1.1, C2.2, C3.2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: now also C5.2, C6.2, C7.2, R13.1, R14.1, R15.1, R16.1, R17.1, R18.1, R19.1, R21.1, R22.1, R23.1, R24.1, R25.1, R26.1, R27.1, R28.1, R29.1, R30.1, R31.1, R32.1, R33.1, R34.1, R35.1, R36.1, U10.11 (COM), U10.9 (GND), U11.11 (COM), U11.9 (GND), U9.11 (COM), U9.9 (GND)
- new net: R35.2, U11.7 (CH6)
- new net: R22.2, U10.2 (CH1)
- new net: C14.1, U12.20 (CPOUT)
- new net: R18.2, U9.6 (CH5)
- new net: C13.1, U12.10 (REGOUT)
- new net: R37.2, U9.10 (REFin/REFout)
- new net: R38.2, U10.10 (REFin/REFout)
- new net: R24.2, U10.4 (CH3)
- new net: R16.2, U9.4 (CH3)
- new net: R32.2, U11.4 (CH3)
- new net: R31.2, U11.3 (CH2)
- new net: R17.2, U9.5 (CH4)
- new net: R29.2, U11.1 (CH0)
- new net: R15.2, U9.3 (CH2)
- new net: R25.2, U10.5 (CH4)
- new net: R13.2, U9.1 (CH0)
- new net: R14.2, U9.2 (CH1)
- new net: R19.2, U9.7 (CH6)
- new net: R20.2, U9.8 (CH7)
- new net: R39.2, U11.10 (REFin/REFout)
- new net: R23.2, U10.3 (CH2)
- new net: R26.2, U10.6 (CH5)
- new net: R30.2, U11.2 (CH1)
- new net: R33.2, U11.5 (CH4)
- new net: R34.2, U11.6 (CH5)
- new net: R36.2, U11.8 (CH7)
- new net: R27.2, U10.7 (CH6)
- new net: R28.2, U10.8 (CH7)
- new net: R21.2, U10.1 (CH0)
- new net +3V3: C10.1, C11.1, C12.1, C9.1, R40.1, R41.1, R42.1, R43.2, R44.2, U12.13 (VDD), U12.8 (VLOGIC), U4.5 (VOUT)
- new net +5V: C8.1, J1.1 (Pin_1), U4.1 (VIN), U4.3 (EN)
- new net AD0: J1.7 (Pin_7), U12.9 (AD0)
- new net GND: C10.2, C11.2, C12.2, C13.2, C14.2, C8.2, C9.2, J1.2 (Pin_2), R40.2, U12.1 (CLKIN), U12.11 (FSYNC), U12.18 (GND), U4.2 (GND)
- new net INT: J1.8 (Pin_8), U12.12 (INT)
- new net SCL: J1.3 (Pin_3), R41.2, U12.23 (SCL)
- new net SDA: J1.4 (Pin_4), R42.2, U12.24 (SDA)
- new net XCL: J1.6 (Pin_6), R44.1, U12.7 (AUX_CL)
- new net XDA: J1.5 (Pin_5), R43.1, U12.6 (AUX_DA)
Other:
- moved on the sheet: C1, C2, C3, C4, D1, D2, D3, MK1, R1, R10, R11, R12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
