File: PCB/Type2 sheet/Sheet.kicad_sch (KiCad schematic)
At the start: 59 parts, among them U1 MCP9700Ax-ELT, U10 ADS7830, U11 ADS7830, U2 MCP2562-E-MF, U3 ATtiny1616-M, U5 CD74HC4067SM, U6 MCP2515-xST, U7 DRV5055A1xDBZxQ1, U8 DRV5055A1xDBZxQ1, U9 ADS7830, Y1 8Mhz

Commit message: new
Parts:
- removed U4: ~, symbol sensors:ADXL335
- added C5, C6, C7: C, symbol Device:C
Connections:
- net at C1.1, C2.2, C3.2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: now also C5.2, C6.2, C7.2
- net at C1.2, C3.1, R37.1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: now also C5.1, C6.1, C7.1

Commit message: sheet with mic
Parts:
- added C10, C11, C12, C13: 0.1uF, Capacitor_SMD:C_0603_1608Metric, symbol Device:C_Small
- added C14: 220pF, Capacitor_SMD:C_0603_1608Metric, symbol Device:C_Small
- added C8: 4.7uF, Capacitor_SMD:C_0603_1608Metric, symbol Device:C_Small
- added C9: 10uF, Capacitor_SMD:C_0603_1608Metric, symbol Device:C_Small
- added J1: Conn_01x08, Connector_PinHeader_2.54mm:PinHeader_1x08_P2.54mm_Horizontal, symbol Connector_Generic:Conn_01x08
- added R40: 1k, Resistor_SMD:R_0603_1608Metric, symbol Device:R_Small_US
- added R41, R42, R43, R44: 4.7k, Resistor_SMD:R_0603_1608Metric, symbol Device:R_Small_US
- added U12: MPU-6050, Sensor_Motion:InvenSense_QFN-24_4x4mm_P0.5mm, symbol Sensor_Motion:MPU-6050
- added U4: AP2112K-3.3, Package_TO_SOT_SMD:SOT-23-5, symbol Regulator_Linear:AP2112K-3.3
Connections:
- new net: C14.1, U12.20 (CPOUT)
- new net: C13.1, U12.10 (REGOUT)
- new net +3V3: C10.1, C11.1, C12.1, C9.1, R40.1, R41.1, R42.1, R43.2, R44.2, U12.13 (VDD), U12.8 (VLOGIC), U4.5 (VOUT)
- new net +5V: C8.1, J1.1 (Pin_1), U4.1 (VIN), U4.3 (EN)
- new net AD0: J1.7 (Pin_7), U12.9 (AD0)
- new net GND: C10.2, C11.2, C12.2, C13.2, C14.2, C8.2, C9.2, J1.2 (Pin_2), R40.2, U12.1 (CLKIN), U12.11 (FSYNC), U12.18 (GND), U4.2 (GND)
- new net INT: J1.8 (Pin_8), U12.12 (INT)
- new net SCL: J1.3 (Pin_3), R41.2, U12.23 (SCL)
- new net SDA: J1.4 (Pin_4), R42.2, U12.24 (SDA)
- new net XCL: J1.6 (Pin_6), R44.1, U12.7 (AUX_CL)
- new net XDA: J1.5 (Pin_5), R43.1, U12.6 (AUX_DA)
Other:
- moved on the sheet: C1, C2, C3, C4, C5, C6, C7, D1, D2, D3, MK1, R1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
