File: PCB/Type2 sheet/Sheet.kicad_pcb (KiCad board)
At the start: 2 copper layers, 139.7 x 49 mm, 46 parts, among them P1 C_0201_0603Metric_Pad0.64x0.4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, U1 MCP9700Ax-ELT, U10 ADS7830, U11 ADS7830, U2 MCP2562-E-MF, U3 ATtiny1616-M, U5 CD74HC4067SM, U6 MCP2515-xST, U7 DRV5055A1xDBZxQ1, U8 DRV5055A1xDBZxQ1, U9 ADS7830

Commit message: updates
Routing:
- net Net-(MK1--): track 18.8 -> 63.6 mm, vias 1 -> 7
- net Net-(U9-CH7): track 0.00 -> 7.52 mm
- net (no net): track 1747.8 -> 1740.6 mm, vias 128 -> 124
- net Net-(U9-CH3): track 18.4 -> 21.7 mm
- net Net-(U9-CH5): track 10.4 -> 13.0 mm
- net Net-(U9-CH2): track 37.2 -> 39.1 mm
- net Net-(U9-CH1): track 18.0 -> 19.5 mm
- net Net-(U9-CH4): track 18.6 -> 19.7 mm

Commit message: new
Parts:
- removed LED4, LED5 (x2): LED_1206_3216Metric, LED_SMD:LED_1206_3216Metric
- added G***1: LOGO, LOGO, F.Cu at (170.8, 47.5)
- added G***2: LOGO, LOGO, F.Cu at (209.7, 113.2)
- added JST1: JST_ACH_BM04B-ACHSS-A-GAN-ETF_1x04-1MP_P1.20mm_Vertical, Connector_JST:JST_ACH_BM04B-ACHSS-A-GAN-ETF_1x04-1MP_P1.20mm_Vertical, F.Cu at (143.1, 85.6)
- added JST1: JST_ACH_BM04B-ACHSS-A-GAN-ETF_1x04-1MP_P1.20mm_Vertical, Connector_JST:JST_ACH_BM04B-ACHSS-A-GAN-ETF_1x04-1MP_P1.20mm_Vertical, F.Cu at (171.4, 112.9)
- added JST2: JST_ACH_BM04B-ACHSS-A-GAN-ETF_1x04-1MP_P1.20mm_Vertical, Connector_JST:JST_ACH_BM04B-ACHSS-A-GAN-ETF_1x04-1MP_P1.20mm_Vertical, F.Cu at (188.7, 79.5)
- added JST2: JST_ACH_BM04B-ACHSS-A-GAN-ETF_1x04-1MP_P1.20mm_Vertical, Connector_JST:JST_ACH_BM04B-ACHSS-A-GAN-ETF_1x04-1MP_P1.20mm_Vertical, F.Cu at (152.0, 81.8)
- added JST3: JST_ACH_BM04B-ACHSS-A-GAN-ETF_1x04-1MP_P1.20mm_Vertical, Connector_JST:JST_ACH_BM04B-ACHSS-A-GAN-ETF_1x04-1MP_P1.20mm_Vertical, F.Cu at (189.5, 70.4)
- added JST4: JST_ACH_BM04B-ACHSS-A-GAN-ETF_1x04-1MP_P1.20mm_Vertical, Connector_JST:JST_ACH_BM04B-ACHSS-A-GAN-ETF_1x04-1MP_P1.20mm_Vertical, F.Cu at (180.5, 117.9)
- added P2: C_0201_0603Metric_Pad0.64x0.40mm_HandSolder, Capacitor_SMD:C_0201_0603Metric_Pad0.64x0.40mm_HandSolder, F.Cu at (182.1, 67.8)
- added P3: C_0201_0603Metric_Pad0.64x0.40mm_HandSolder, Capacitor_SMD:C_0201_0603Metric_Pad0.64x0.40mm_HandSolder, F.Cu at (182.8, 67.4)
- added P4: C_0201_0603Metric_Pad0.64x0.40mm_HandSolder, Capacitor_SMD:C_0201_0603Metric_Pad0.64x0.40mm_HandSolder, F.Cu at (186.5, 112.8)
- added P5: C_0201_0603Metric_Pad0.64x0.40mm_HandSolder, Capacitor_SMD:C_0201_0603Metric_Pad0.64x0.40mm_HandSolder, F.Cu at (186.5, 113.6)
- added R22: R, Resistor_SMD:R_0201_0603Metric, F.Cu at (157.2, 71.2)
- added R23: R, Resistor_SMD:R_0201_0603Metric, F.Cu at (164.6, 50.5)
- added R24: R, Resistor_SMD:R_0201_0603Metric, F.Cu at (167.3, 60.6)
- added R25: R, Resistor_SMD:R_0201_0603Metric, F.Cu at (174.1, 61.9)
- added R26: R, Resistor_SMD:R_0201_0603Metric, F.Cu at (194.2, 70.0)
- added R27: R, Resistor_SMD:R_0201_0603Metric, F.Cu at (181.8, 60.1)
- added R28: R, Resistor_SMD:R_0201_0603Metric, F.Cu at (179.9, 48.8)
- added R29: R, Resistor_SMD:R_0201_0603Metric, F.Cu at (175.6, 46.0)
- added R30: R, Resistor_SMD:R_0201_0603Metric, F.Cu at (174.7, 36.8)
- added R31: R, Resistor_SMD:R_0201_0603Metric, F.Cu at (196.0, 89.6)
- added R32: R, Resistor_SMD:R_0201_0603Metric, F.Cu at (210.3, 106.4)
- added R33: R, Resistor_SMD:R_0201_0603Metric, F.Cu at (200.1, 103.7)
- added R34: R, Resistor_SMD:R_0201_0603Metric, F.Cu at (195.6, 108.9)
- added R35: R, Resistor_SMD:R_0201_0603Metric, F.Cu at (178.5, 122.3)
- added R36: R, Resistor_SMD:R_0201_0603Metric, F.Cu at (193.3, 116.5)
- added R38: R, Resistor_SMD:R_0201_0603Metric, F.Cu at (177.1, 65.7)
- added R39: R, Resistor_SMD:R_0201_0603Metric, F.Cu at (204.1, 120.4)
- added R40: R, Resistor_SMD:R_0201_0603Metric, F.Cu at (208.7, 118.2)
- added R41: R, Resistor_SMD:R_0201_0603Metric, F.Cu at (217.1, 121.9)
- added R42: R, Resistor_SMD:R_0201_0603Metric, F.Cu at (190.8, 109.5)
- added RP5: 10K Pack, RESPACK_4X0603, F.Cu at (184.7, 61.1)
- added RP6: 10K Pack, RESPACK_4X0603, F.Cu at (191.0, 118.4)
- moved U11 106.1 mm to (191.7, 113.0), turned to 180 degrees
- moved U10 94.6 mm to (179.6, 63.1), turned to -60 degrees
- moved R13 69.6 mm to (159.9, 113.2), turned to 60 degrees
- moved R14 66.3 mm to (138.2, 117.2), turned to 60 degrees
- moved R21 63.7 mm to (121.4, 115.3), turned to 60 degrees
- moved G*** 61.7 mm to (132.6, 113.3), turned to 60 degrees
- moved R15 60.8 mm to (145.7, 109.8), turned to 60 degrees
- moved R20 58.1 mm to (128.8, 109.9), turned to 60 degrees
- moved R16 54.0 mm to (143.4, 103.3), turned to 60 degrees
- moved R19 53.0 mm to (129.1, 104.8), turned to 60 degrees
- moved R37 50.3 mm to (145.2, 98.8), turned to 60 degrees
- moved U9 48.4 mm to (141.7, 98.0), turned to 60 degrees
- moved P1 45.1 mm to (144.5, 93.4), turned to 60 degrees
- moved R18 45.0 mm to (138.0, 97.5), turned to 60 degrees
- moved P1 44.5 mm to (143.8, 93.0), turned to 60 degrees
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Routing:
- net (no net): track 1740.6 -> 3075.1 mm, vias 124 -> 190
- net Net-(MK1--): track 63.6 -> 491.8 mm, vias 7 -> 47
- net Net-(U1-V_{DD}): track 162.7 -> 456.8 mm, vias 16 -> 54
- net Net-(U9-CH0): track 6.75 -> 136.0 mm, vias 0 -> 7
- net Net-(U10-SDA): track 25.6 -> 102.3 mm, vias 3 -> 11
- net Net-(U10-CH0): track 0.00 -> 75.5 mm, vias 0 -> 3
- net Net-(U10-SCL): track 15.2 -> 86.5 mm, vias 2 -> 11
- net unconnected-(R20-Pad1): track 0.00 -> 39.0 mm, vias 0 -> 4
- net Net-(U9-CH1): track 19.5 -> 51.0 mm
- net Net-(U9-CH5): track 13.0 -> 32.7 mm, vias 1 -> 4
- net Net-(U9-CH4): track 19.7 -> 38.3 mm
- net Net-(U4-XOUT): track 14.4 -> 0.14 mm
- net unconnected-(U10-A0-Pad12): track 0.00 -> 12.0 mm, vias 0 -> 2
- net unconnected-(U11-A0-Pad12): track 0.00 -> 12.0 mm, vias 0 -> 2
- net unconnected-(U11-A1-Pad13): track 0.00 -> 10.4 mm
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Other:
- board size 139.7 x 49 mm -> 113 x 97.3 mm

Commit message: Update Sheet.kicad_pcb
Parts:
- moved R11 2.23 mm to (193.4, 78.9), turned to 90 degrees
- moved R34 1.16 mm to (194.7, 108.2)
- moved R40 1.16 mm to (207.7, 117.4)
- moved JST4 1.16 mm to (179.6, 117.2)
- moved P4 1.16 mm to (185.6, 112.1)
- moved P5 1.16 mm to (185.6, 112.9)
- moved R32 1.16 mm to (209.3, 105.7)
- moved R36 1.16 mm to (192.4, 115.8)
- moved R41 1.16 mm to (216.1, 121.2)
- moved R42 1.16 mm to (189.9, 108.8)
- moved RP6 1.16 mm to (190.1, 117.7)
- moved U11 1.16 mm to (190.7, 112.3)
- moved G***2 1.16 mm to (208.8, 112.5)
- moved R31 1.16 mm to (195.1, 88.9)
- moved R33 1.16 mm to (199.2, 103.0)
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- renumbered JST1 to JST2, JST1 to JSTA, JST2 to JSTB, JST2 to JSTC
Routing:
- net Net-(U10-SCL): track 86.5 -> 196.9 mm, vias 11 -> 25
- net Net-(U5-I1): track 0.00 -> 84.5 mm, vias 0 -> 7
- net Net-(U5-I7): track 17.7 -> 74.2 mm, vias 1 -> 14
- net Net-(U5-I5): track 34.3 -> 88.6 mm, vias 3 -> 9
- net (no net): track 3075.1 -> 3022.7 mm, vias 190 -> 182
- net Net-(U1-V_{DD}): track 456.8 -> 472.8 mm, vias 54 -> 56
- net Net-(U10-SDA): track 102.3 -> 113.3 mm, vias 11 -> 10
- net Net-(MK1--): track 491.8 -> 495.7 mm
- net Net-(U2-CANH): track 162.8 -> 163.8 mm
- net Net-(U3-PB5): track 31.8 -> 31.3 mm
Other:
- board size 113 x 97.3 mm -> 111.2 x 96.9 mm

Commit message: sheet with mic
Parts:
- removed the P1 at (144.7, 93.0)
- removed the P1 at (145.4, 93.4)
- added C10: 0.1uF, Capacitor_SMD:C_0603_1608Metric, F.Cu at (218.0, 103.4)
- added C12: 0.1uF, Capacitor_SMD:C_0603_1608Metric, F.Cu at (229.1, 103.4)
- added C13: 0.1uF, Capacitor_SMD:C_0603_1608Metric, F.Cu at (229.9, 105.6)
- added C14: 220pF, Capacitor_SMD:C_0603_1608Metric, F.Cu at (218.6, 105.8)
- added C8: 4.7uF, Capacitor_SMD:C_0603_1608Metric, F.Cu at (215.1, 109.8)
- added P1: C_0201_0603Metric_Pad0.64x0.40mm_HandSolder, Capacitor_SMD:C_0201_0603Metric_Pad0.64x0.40mm_HandSolder, F.Cu at (179.7, 119.9)
- added P1: C_0201_0603Metric_Pad0.64x0.40mm_HandSolder, Capacitor_SMD:C_0201_0603Metric_Pad0.64x0.40mm_HandSolder, F.Cu at (180.4, 120.3)
- added R43: 4.7k, Resistor_SMD:R_0603_1608Metric, F.Cu at (228.6, 109.3)
- added R44: 4.7k, Resistor_SMD:R_0603_1608Metric, F.Cu at (224.4, 115.2)
- added R9: R9, Resistor_SMD:R_0201_0603Metric, F.Cu at (198.8, 133.6)
- added REF**: PinHeader_1x02_P1.00mm_Vertical, Connector_PinHeader_1.00mm:PinHeader_1x02_P1.00mm_Vertical, F.Cu at (200.6, 133.2)
- added U12: MPU-6050, Sensor_Motion:InvenSense_QFN-24_4x4mm_P0.5mm, F.Cu at (224.5, 111.8)
- added U4: AP2112K-3.3, Package_TO_SOT_SMD:SOT-23-5, F.Cu at (215.3, 107.2)
- R40: value R -> 1k
- R41, R42: value R -> 4.7k
- moved R20 44.2 mm to (164.8, 136.8)
- moved G*** 44.2 mm to (168.5, 140.2)
- moved JST2 44.2 mm to (179.0, 112.5)
- moved R18 44.2 mm to (173.9, 124.3)
- moved R21 44.2 mm to (157.3, 142.2)
- moved R37 44.2 mm to (181.1, 125.6)
- moved RP4 44.2 mm to (173.3, 121.3)
- moved U9 44.2 mm to (177.6, 124.8)
- moved R13 44.2 mm to (195.8, 140.1)
- moved R14 44.2 mm to (174.2, 144.1)
- moved R16 44.2 mm to (179.3, 130.1)
- moved R19 44.2 mm to (165.1, 131.7)
- moved R15 44.2 mm to (181.6, 136.6)
- moved R17 44.2 mm to (176.3, 108.6)
- moved P4 44.2 mm to (220.6, 139.0)
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Connections:
- R22 pad 2: Net-(U9-CH0) -> Net-(U10-CH1)
- R23 pad 2: Net-(U9-CH1) -> Net-(U10-CH2)
- R24 pad 2: Net-(U9-CH2) -> Net-(U10-CH3)
- R25 pad 2: Net-(U9-CH3) -> Net-(U10-CH4)
- R26 pad 2: Net-(U9-CH4) -> Net-(U10-CH5)
- R27 pad 2: Net-(U9-CH5) -> Net-(U10-CH6)
- R28 pad 2: Net-(U9-CH6) -> Net-(U10-CH7)
- R29 pad 1: unconnected-(R20-Pad1) -> Net-(MK1--)
- R29 pad 2: Net-(U9-CH7) -> Net-(U11-CH0)
- R30 pad 2: Net-(U10-CH0) -> Net-(U11-CH1)
- R31 pad 2: Net-(U9-CH0) -> Net-(U11-CH2)
- R32 pad 2: Net-(U9-CH1) -> Net-(U11-CH3)
- R33 pad 2: Net-(U9-CH2) -> Net-(U11-CH4)
- R34 pad 2: Net-(U9-CH3) -> Net-(U11-CH5)
- R35 pad 2: Net-(U9-CH4) -> Net-(U11-CH6)
- R36 pad 2: Net-(U9-CH5) -> Net-(U11-CH7)
- R38 pad 2: Net-(U9-REFin/REFout) -> Net-(U10-REFin/REFout)
- R39 pad 1: Net-(MK1--) -> Net-(U1-V_{DD})
- R39 pad 2: Net-(U9-CH6) -> Net-(U11-REFin/REFout)
- R40 pad 1: unconnected-(R20-Pad1) -> +3V3
- R40 pad 2: Net-(U9-CH7) -> Net-(D4-A)
- R41 pad 1: Net-(MK1--) -> +3V3
- R41 pad 2: Net-(U10-CH0) -> /SCL
- R42 pad 1: Net-(U1-V_{DD}) -> +3V3
- R42 pad 2: Net-(U9-REFin/REFout) -> /SDA
- U5 pad 18: Net-(U4-ZOUT) -> unconnected-(U5-I13-Pad18)
- U5 pad 21: Net-(U4-YOUT) -> unconnected-(U5-I10-Pad21)
- U5 pad 22: Net-(U4-XOUT) -> unconnected-(U5-I9-Pad22)
Routing:
- net (no net): track 3022.7 -> 2905.6 mm, vias 182 -> 183
- net Net-(U11-CH2): track 0.00 -> 52.8 mm, vias 0 -> 2
- net +3V3: track 0.00 -> 41.6 mm, vias 0 -> 4
- net Net-(U11-CH1): track 0.00 -> 33.2 mm, vias 0 -> 2
- net Net-(MK1--): track 495.7 -> 464.2 mm, vias 47 -> 45
- net Net-(U11-CH7): track 0.00 -> 22.7 mm, vias 0 -> 1
- net Net-(U1-V_{DD}): track 472.8 -> 493.2 mm, vias 56 -> 58
- net unconnected-(R20-Pad1): track 39.0 -> 19.5 mm, vias 4 -> 2
- net GND: track 0.00 -> 15.0 mm
- net Net-(U5-I5): track 88.6 -> 102.4 mm
- net Net-(U5-I14): track 11.7 -> 25.5 mm
- net Net-(U5-I12): track 16.9 -> 30.7 mm
- net Net-(U5-I1): track 84.5 -> 97.3 mm, vias 7 -> 8
- net Net-(U5-I6): track 19.5 -> 31.6 mm
- net Net-(U12-REGOUT): track 0.00 -> 10.4 mm, vias 0 -> 2
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Other:
- outline, holes or cut-outs redrawn

Commit message: sheet usable
Parts:
- removed crystal: Crystal_SMD_2012-2Pin_2.0x1.2mm, Crystal:Crystal_SMD_2012-2Pin_2.0x1.2mm
- added CRYSTAL: Crystal 8MHz, Connector_PinHeader_1.27mm:PinHeader_2x01_P1.27mm_Vertical, F.Cu at (200.2, 104.8)
- R40: value 1k -> R
- R41: value 4.7k -> R
Routing:
- net Net-(MK1--): track 464.2 -> 530.0 mm, vias 45 -> 49
- net Net-(U5-I1): track 97.3 -> 35.9 mm, vias 8 -> 4
- net Net-(U1-V_{DD}): track 493.2 -> 499.0 mm
- net (no net): track 2905.6 -> 2907.1 mm
- net Net-(U9-CH0): track 136.0 -> 136.8 mm
- net Net-(U10-SCL): track 196.9 -> 197.5 mm
Other:
- board size 111.2 x 96.9 mm -> 111.3 x 96.9 mm

Commit message: fixes for manufacturing
Parts:
- removed the CRYSTAL at (200.2, 104.8)
- added CRYSTAL: Crystal_HC52-6mm_Vertical, Crystal:Crystal_HC52-6mm_Vertical, F.Cu at (194.7, 104.8)
- R42: value 4.7k -> R
- moved JST4 0.50 mm to (214.5, 144.6)
- moved P5 0.50 mm to (220.5, 140.3)
- moved R32 0.50 mm to (244.2, 133.0)
- moved P4 0.50 mm to (220.5, 139.5)
- moved R33 0.50 mm to (234.1, 130.3)
- moved R40 0.50 mm to (242.6, 144.8)
- moved R34 0.50 mm to (229.6, 135.6)
- moved R41 0.50 mm to (251.0, 148.6)
- moved R35 0.50 mm to (212.5, 148.9)
- moved R39 0.50 mm to (238.1, 147.1)
- moved RP6 0.50 mm to (225.0, 145.1)
- moved R36 0.50 mm to (227.3, 143.1)
- moved R42 0.50 mm to (224.8, 136.2)
- moved G***2 0.50 mm to (243.7, 139.8)
- moved R31 0.50 mm to (230.0, 116.2)
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Connections:
- R22 pad 2: Net-(U10-CH1) -> Net-(U9-CH0)
- R23 pad 2: Net-(U10-CH2) -> Net-(U9-CH1)
- R24 pad 2: Net-(U10-CH3) -> Net-(U9-CH2)
- R25 pad 2: Net-(U10-CH4) -> Net-(U9-CH3)
- R26 pad 2: Net-(U10-CH5) -> Net-(U9-CH4)
- R27 pad 2: Net-(U10-CH6) -> Net-(U9-CH5)
- R28 pad 2: Net-(U10-CH7) -> Net-(U9-CH6)
- R29 pad 1: Net-(MK1--) -> unconnected-(R20-Pad1)
- R29 pad 2: Net-(U11-CH0) -> Net-(U9-CH7)
- R30 pad 2: Net-(U11-CH1) -> Net-(U10-CH0)
- R31 pad 2: Net-(U11-CH2) -> Net-(U9-CH0)
- R32 pad 2: Net-(U11-CH3) -> Net-(U9-CH1)
- R33 pad 2: Net-(U11-CH4) -> Net-(U9-CH2)
- R34 pad 2: Net-(U11-CH5) -> Net-(U9-CH3)
- R35 pad 2: Net-(U11-CH6) -> Net-(U9-CH4)
- R36 pad 2: Net-(U11-CH7) -> Net-(U9-CH5)
- R38 pad 2: Net-(U10-REFin/REFout) -> Net-(U9-REFin/REFout)
- R39 pad 1: Net-(U1-V_{DD}) -> Net-(MK1--)
- R39 pad 2: Net-(U11-REFin/REFout) -> Net-(U9-CH6)
- R40 pad 1: +3V3 -> unconnected-(R20-Pad1)
- R40 pad 2: Net-(D4-A) -> Net-(U9-CH7)
- R41 pad 1: +3V3 -> Net-(MK1--)
- R41 pad 2: /SCL -> Net-(U10-CH0)
- R42 pad 1: +3V3 -> Net-(U1-V_{DD})
- R42 pad 2: /SDA -> Net-(U9-REFin/REFout)
- U10 pad 1: Net-(U10-CH0) -> Net-(U9-CH0)
- U10 pad 10: Net-(U10-REFin/REFout) -> Net-(U9-REFin/REFout)
- U10 pad 12: unconnected-(U10-A0-Pad12) -> unconnected-(U9-A0-Pad12)
- U10 pad 13: unconnected-(U10-A1-Pad13) -> unconnected-(U9-A1-Pad13)
- U10 pad 2: Net-(U10-CH1) -> Net-(U9-CH1)
- U10 pad 3: Net-(U10-CH2) -> Net-(U9-CH2)
- U10 pad 4: Net-(U10-CH3) -> Net-(U9-CH3)
- U10 pad 5: Net-(U10-CH4) -> Net-(U9-CH4)
- U10 pad 6: Net-(U10-CH5) -> Net-(U9-CH5)
- U10 pad 7: Net-(U10-CH6) -> Net-(U9-CH6)
- U10 pad 8: Net-(U10-CH7) -> Net-(U9-CH7)
- U11 pad 1: Net-(U11-CH0) -> Net-(U9-CH0)
- U11 pad 10: Net-(U11-REFin/REFout) -> Net-(U9-REFin/REFout)
- U11 pad 12: unconnected-(U11-A0-Pad12) -> unconnected-(U9-A0-Pad12)
- U11 pad 13: unconnected-(U11-A1-Pad13) -> unconnected-(U9-A1-Pad13)
- U11 pad 2: Net-(U11-CH1) -> Net-(U9-CH1)
- U11 pad 3: Net-(U11-CH2) -> Net-(U9-CH2)
- U11 pad 4: Net-(U11-CH3) -> Net-(U9-CH3)
- U11 pad 5: Net-(U11-CH4) -> Net-(U9-CH4)
- U11 pad 6: Net-(U11-CH5) -> Net-(U9-CH5)
- U11 pad 7: Net-(U11-CH6) -> Net-(U9-CH6)
- U11 pad 8: Net-(U11-CH7) -> Net-(U9-CH7)
Routing:
- net (no net): track 2907.1 -> 1211.9 mm, vias 183 -> 74
- net Net-(MK1--): track 530.0 -> 1216.2 mm, vias 49 -> 64
- net Net-(U1-V_{DD}): track 499.0 -> 1055.6 mm, vias 58 -> 120
- net Net-(U2-CANL): track 0.00 -> 326.2 mm, vias 0 -> 32
- net Net-(U9-CH2): track 39.1 -> 117.3 mm, vias 2 -> 6
- net Net-(U11-CH2): track 52.8 -> 0.00 mm, vias 2 -> 0
- net Net-(U9-CH3): track 21.7 -> 65.1 mm, vias 2 -> 6
- net Net-(U9-CH4): track 38.3 -> 77.7 mm, vias 1 -> 3
- net Net-(U9-CH1): track 51.0 -> 90.0 mm, vias 2 -> 6
- net Net-(U11-CH1): track 33.2 -> 0.00 mm, vias 2 -> 0
- net Net-(U9-CH0): track 136.8 -> 166.8 mm, vias 7 -> 9
- net Net-(U2-RXD): track 0.00 -> 29.1 mm, vias 0 -> 2
- net unconnected-(U9-A0-Pad12): track 12.0 -> 36.0 mm, vias 2 -> 6
- net Net-(U11-CH7): track 22.7 -> 0.00 mm, vias 1 -> 0
- net unconnected-(U9-A1-Pad13): track 10.4 -> 31.1 mm
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Other:
- board size 111.3 x 96.9 mm -> 111 x 97.1 mm
